Commit message: fixed code and finished actions

File: SPRING_2025/Intro To Robotics/MODULE_5/class4_ws/install/en613_control/share/en613_control/urdf/basic_robot.urdf (robot description, URDF)
Before this commit: robot basic_robot, 4 links, 3 joints
Links:
- link chassis: mass None -> 10.0
Joints:
- joint chassis_to_left_wheel: axis 0 1 0 -> 0 0 1; origin xyz=0 0 0 -> xyz=0 0.4375 0 rpy=-1.5708 0 0
- joint chassis_to_lidar_dome: origin xyz=0 0 0 -> xyz=0.3 0 0.0375 rpy=0 0 0
- joint chassis_to_right_wheel: axis 0 1 0 -> 0 0 1; origin xyz=0 0 0 -> xyz=0 -0.4375 0 rpy=1.5708 0 0

Commit message: Edited out inertial from chassis

File: SPRING_2025/Intro To Robotics/MODULE_5/class4_ws/install/en613_control/share/en613_control/urdf/basic_robot.urdf (robot description, URDF)
Before this commit: robot basic_robot, 4 links, 3 joints
Links:
- link chassis: mass 10.0 -> None
